Commit message: updated all the functionality with speech recognision

File: bernado_description/robots/inmoov.urdf (robot description, URDF)
Before this commit: robot inmoov, 25 links, 24 joints
Links:
- link chestplate: geometry visual mesh filename=package://chest.dae scale=0.001 0.001 0.001
- link disk: geometry visual mesh filename=package://disk.dae scale=0.001 0.001 0.001
- link eyesupport: geometry visual mesh filename=package://eyesupport.dae scale=0.001 0.001 0.001
- link face: geometry visual mesh filename=package://face.dae scale=0.001 0.001 0.001
- link head: geometry visual mesh filename=package://head.dae scale=0.001 0.001 0.001
- link head_base: geometry visual mesh filename=package://head_base.dae scale=0.001 0.001 0.001
- link head_tilt: geometry visual mesh filename=package://virtual.dae scale=0.001 0.001 0.001
- link jaw: geometry visual mesh filename=package://jaw.dae scale=0.001 0.001 0.001
- link kinect: geometry visual mesh filename=package://kinectone.dae scale=0.001 0.001 0.001
- link left_bicep: geometry visual mesh filename=package://bicep.dae scale=0.001 0.001 0.001
- link left_ear: geometry visual mesh filename=package://earleftv1.dae scale=0.001 0.001 0.001
- link left_forearm: geometry visual mesh filename=package://left_forearm.dae scale=0.001 0.001 0.001
- link left_shoulder: geometry visual mesh filename=package://left_shoulder.dae scale=0.001 0.001 0.001
- link left_shoulder_base: geometry visual mesh filename=package://left_shoulder_base.dae scale=0.001 0.001 0.001
- link mid_stomach: geometry visual mesh filename=package://mid_stomach.dae scale=0.001 0.001 0.001
- link right_bicep: geometry visual mesh filename=package://bicep.dae scale=0.001 0.001 0.001
- link right_ear: geometry visual mesh filename=package://earrightv1.dae scale=0.001 0.001 0.001
- link right_forearm: geometry visual mesh filename=package://right_forearm.dae scale=0.001 0.001 0.001
- link right_shoulder: geometry visual mesh filename=package://right_shoulder.dae scale=0.001 0.001 0.001
- link right_shoulder_base: geometry visual mesh filename=package://right_shoulder_base.dae scale=0.001 0.001 0.001
- link skull: geometry visual mesh filename=package://skull.dae scale=0.001 0.001 0.001
- link top_stomach: geometry visual mesh filename=package://top_stomach.dae scale=0.001 0.001 0.001
- link torso: geometry visual mesh filename=package://torso.dae scale=0.001 0.001 0.001

Commit message: updated speech localization

File: bernado_description/robots/inmoov.urdf (robot description, URDF)
Before this commit: robot inmoov, 25 links, 24 joints
Links:
- link chestplate: geometry visual mesh filename=file:///home/viki/Desktop/bernado_ros/bernado_description/m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 scale=0.001 0.001 0.001
- link disk: geometry visual mesh filename=file:///home/viki/Desktop/bernado_ros/bernado_description/m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 scale=0.001 0.001 0.001
- link eyesupport: geometry visual mesh filename=file:///home/viki/Desktop/bernado_ros/bernado_description/m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 scale=0.001 0.001 0.001
- link face: geometry visual mesh filename=file:///home/viki/Desktop/bernado_ros/bernado_description/m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 scale=0.001 0.001 0.001
- link head: geometry visual mesh filename=file:///home/viki/Desktop/bernado_ros/bernado_description/m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 scale=0.001 0.001 0.001
- link head_base: geometry visual mesh filename=file:///home/viki/Desktop/bernado_ros/bernado_description/m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 scale=0.001 0.001 0.001
- link head_tilt: geometry visual mesh filename=file:///home/viki/Desktop/bernado_ros/bernado_description/m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 scale=0.001 0.001 0.001
- link jaw: geometry visual mesh filename=file:///home/viki/Desktop/bernado_ros/bernado_description/m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 scale=0.001 0.001 0.001
- link kinect: geometry visual mesh filename=file:///home/viki/Desktop/bernado_ros/bernado_description/m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 scale=0.001 0.001 0.001
- link left_bicep: geometry visual mesh filename=file:///home/viki/Desktop/bernado_ros/bernado_description/m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 scale=0.001 0.001 0.001
- link left_ear: geometry visual mesh filename=file:///home/viki/Desktop/bernado_ros/bernado_description/m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 scale=0.001 0.001 0.001
- link left_forearm: geometry visual mesh filename=file:///home/viki/Desktop/bernado_ros/bernado_description/m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 scale=0.001 0.001 0.001
- link left_shoulder: geometry visual mesh filename=file:///home/viki/Desktop/bernado_ros/bernado_description/m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 scale=0.001 0.001 0.001
- link left_shoulder_base: geometry visual mesh filename=file:///home/viki/Desktop/bernado_ros/bernado_description/m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 scale=0.001 0.001 0.001
- link mid_stomach: geometry visual mesh filename=file:///home/viki/Desktop/bernado_ros/bernado_description/m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 scale=0.001 0.001 0.001
- link right_bicep: geometry visual mesh filename=file:///home/viki/Desktop/bernado_ros/bernado_description/m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 scale=0.001 0.001 0.001
- link right_ear: geometry visual mesh filename=file:///home/viki/Desktop/bernado_ros/bernado_description/m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 scale=0.001 0.001 0.001
- link right_forearm: geometry visual mesh filename=file:///home/viki/Desktop/bernado_ros/bernado_description/m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 scale=0.001 0.001 0.001
- link right_shoulder: geometry visual mesh filename=file:///home/viki/Desktop/bernado_ros/bernado_description/m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 scale=0.001 0.001 0.001
- link right_shoulder_base: geometry visual mesh filename=file:///home/viki/Desktop/bernado_ros/bernado_description/m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 scale=0.001 0.001 0.001
- link skull: geometry visual mesh filename=file:///home/viki/Desktop/bernado_ros/bernado_description/m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 scale=0.001 0.001 0.001
- link top_stomach: geometry visual mesh filename=file:///home/viki/Desktop/bernado_ros/bernado_description/m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 scale=0.001 0.001 0.001
- link torso: geometry visual mesh filename=file:///home/viki/Desktop/bernado_ros/bernado_description/m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 scale=0.001 0.001 0.001
